File: LED.kicad_sch (KiCad schematic)
At the start: 160 parts, among them Q1 NMOS, Q2 NMOS, Q3 NMOS, Q4 NMOS, Q5 NMOS, Q6 NMOS, Q7 NMOS, U1 74HC574, U2 74HC574, U3 74HC574, U4 74HC574, U5 74HC164

Commit message: Updated the Schematic
Connections:
- net at D64.1 (K), D65.1 (K), D66.1 (K)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: now also D68.1 (K), D69.1 (K), D70.1 (K); no longer D60.1 (K), D62.1 (K), D63.1 (K)
- net at D100.1 (K), D102.1 (K), D103.1 (K)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: now also D101.1 (K), D105.1 (K); no longer D97.1 (K), D98.1 (K)
- net at D53.1 (K), D54.1 (K), D55.1 (K)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: now also D50.1 (K), D51.1 (K), D52.1 (K), U2.16 (Q3); no longer D57.1 (K), D58.1 (K), D59.1 (K), U2.15 (Q4)
- net at D31.1 (K), D32.1 (K), D33.1 (K)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: now also D29.1 (K), D30.1 (K), U1.14 (Q5); no longer D36.1 (K), D37.1 (K), U2.18 (Q1)
- net at D120.1 (K), D122.1 (K), D123.1 (K)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: now also D121.1 (K); no longer D119.1 (K)
- net at D78.1 (K), D79.1 (K), D80.1 (K)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: now also D81.1 (K), D83.1 (K), D84.1 (K); no longer D75.1 (K), D76.1 (K), D77.1 (K)
- net at D71.1 (K), D72.1 (K), D73.1 (K)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: now also D75.1 (K), D76.1 (K), D77.1 (K); no longer D68.1 (K), D69.1 (K), D70.1 (K)
- net at D10.1 (K), D11.1 (K), D12.1 (K)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: now also D8.1 (K), U1.17 (Q2); no longer D15.1 (K), U1.16 (Q3)
- net at D43.1 (K), D44.1 (K), D45.1 (K)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: now also D46.1 (K), D47.1 (K), D48.1 (K), D49.1 (K); no longer D38.1 (K), D39.1 (K), D40.1 (K), D42.1 (K)
- net at D113.1 (K), D114.1 (K), D115.1 (K)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: now also D119.1 (K); no longer D112.1 (K)
- net at D16.1 (K), D17.1 (K), D18.1 (K)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: now also D15.1 (K), D21.1 (K), U1.16 (Q3); no longer D22.1 (K), D23.1 (K), U1.15 (Q4)
- net at D92.1 (K), D93.1 (K), D94.1 (K)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: now also D97.1 (K), D98.1 (K); no longer D90.1 (K), D91.1 (K)
- net at D24.1 (K), D25.1 (K), D26.1 (K)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: now also D22.1 (K), D23.1 (K), U1.15 (Q4); no longer D29.1 (K), D30.1 (K), U1.14 (Q5)
- net at D2.1 (K), D3.1 (K), D4.1 (K)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: now also D1.1 (K), U1.18 (Q1); no longer D8.1 (K), U1.17 (Q2)
- net at D106.1 (K), D107.1 (K), D108.1 (K)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: now also D112.1 (K); no longer D105.1 (K)
- net at D85.1 (K), D86.1 (K), D87.1 (K)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: now also D90.1 (K), D91.1 (K); no longer D83.1 (K), D84.1 (K)
- new net: D102.2 (A), D109.2 (A), D11.2 (A), D116.2 (A), D123.2 (A), D130.2 (A), D137.2 (A), D18.2 (A), D25.2 (A), D32.2 (A), D39.2 (A), D4.2 (A), D46.2 (A), D53.2 (A), D60.2 (A), D67.2 (A), D74.2 (A), D81.2 (A), D88.2 (A), D95.2 (A), Q4.1 (D), R4.2
- new net: D103.2 (A), D110.2 (A), D117.2 (A), D12.2 (A), D124.2 (A), D131.2 (A), D138.2 (A), D19.2 (A), D26.2 (A), D33.2 (A), D40.2 (A), D47.2 (A), D5.2 (A), D54.2 (A), D61.2 (A), D68.2 (A), D75.2 (A), D82.2 (A), D89.2 (A), D96.2 (A), Q5.1 (D), R5.2
- new net: D10.2 (A), D101.2 (A), D108.2 (A), D115.2 (A), D122.2 (A), D129.2 (A), D136.2 (A), D17.2 (A), D24.2 (A), D3.2 (A), D31.2 (A), D38.2 (A), D45.2 (A), D52.2 (A), D59.2 (A), D66.2 (A), D73.2 (A), D80.2 (A), D87.2 (A), D94.2 (A), Q3.1 (D), R3.2
- new net: D1.2 (A), D106.2 (A), D113.2 (A), D120.2 (A), D127.2 (A), D134.2 (A), D15.2 (A), D22.2 (A), D29.2 (A), D36.2 (A), D43.2 (A), D50.2 (A), D57.2 (A), D64.2 (A), D71.2 (A), D78.2 (A), D8.2 (A), D85.2 (A), D92.2 (A), D99.2 (A), Q1.1 (D), R1.2
- new net: D105.2 (A), D112.2 (A), D119.2 (A), D126.2 (A), D133.2 (A), D14.2 (A), D140.2 (A), D21.2 (A), D28.2 (A), D35.2 (A), D42.2 (A), D49.2 (A), D56.2 (A), D63.2 (A), D7.2 (A), D70.2 (A), D77.2 (A), D84.2 (A), D91.2 (A), D98.2 (A), Q7.1 (D), R7.2
- new net: D100.2 (A), D107.2 (A), D114.2 (A), D121.2 (A), D128.2 (A), D135.2 (A), D16.2 (A), D2.2 (A), D23.2 (A), D30.2 (A), D37.2 (A), D44.2 (A), D51.2 (A), D58.2 (A), D65.2 (A), D72.2 (A), D79.2 (A), D86.2 (A), D9.2 (A), D93.2 (A), Q2.1 (D), R2.2
- new net: D104.2 (A), D111.2 (A), D118.2 (A), D125.2 (A), D13.2 (A), D132.2 (A), D139.2 (A), D20.2 (A), D27.2 (A), D34.2 (A), D41.2 (A), D48.2 (A), D55.2 (A), D6.2 (A), D62.2 (A), D69.2 (A), D76.2 (A), D83.2 (A), D90.2 (A), D97.2 (A), Q6.1 (D), R6.2
- new net: D57.1 (K), D58.1 (K), D59.1 (K), D60.1 (K), D61.1 (K), D62.1 (K), D63.1 (K), U2.15 (Q4)
- new net: D36.1 (K), D37.1 (K), D38.1 (K), D39.1 (K), D40.1 (K), D41.1 (K), D42.1 (K), U2.18 (Q1)
